File: Hardware/remote_shutter_controller/mcu.kicad_sch (KiCad schematic)
At the start: 27 parts

Commit message: Schematic updates. First export to PCB
Added 9V line, OLED switch circuit. Added OLED footprint.
Parts:
- removed J?: Buzzer, Connector_PinSocket_2.54mm:PinSocket_1x02_P2.54mm_Vertical, symbol Connector:Conn_01x02_Male
- removed R?: 100, Resistor_SMD:R_0603_1608Metric_Pad0.98x0.95mm_HandSolder, symbol Device:R_Small
- added C5, C6: 0u1, Capacitor_SMD:C_0603_1608Metric_Pad1.08x0.95mm_HandSolder, symbol Device:C_Small
- added S3, S4: 4-1437565-2, footprint:SW_4-1437565-2, symbol 4-1437565-2:4-1437565-2
- gave numbers to parts that had none: 25
Connections:
- net FTRIG: now also C6.1, S4.3, S4.4
- net GND: now also C5.2, C6.2, S3.1, S3.2, S4.1, S4.2
- net STRIG: now also C5.1, S3.3, S3.4
- net DIS_EN: now reaches U1.28 (IO8)
Other:
- sheet Interfaces ports: added 9V, DIS_EN; removed FTRIG, STRIG
- moved on the sheet: C1, C2, C3, C4, R3, R4, S1, S2

Commit message: Layout pre-routing
Parts:
- removed C5, C6: 0u1, Capacitor_SMD:C_0603_1608Metric_Pad1.08x0.95mm_HandSolder, symbol Device:C_Small
- removed S3, S4: 4-1437565-2, footprint:SW_4-1437565-2, symbol 4-1437565-2:4-1437565-2
Changed lines of the file:
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@@
   (junction (at 80.01 167.64) (diameter 0) (color 0 0 0 0)
   )
-  (junction (at 109.22 167.64) (diameter 0) (color 0 0 0 0)
-  )
-  (junction (at 127 134.62) (diameter 0) (color 0 0 0 0)
-  )
   (junction (at 63.5 166.37) (diameter 0) (color 0 0 0 0)
   )
@@
   (junction (at 182.88 57.15) (diameter 0) (color 0 0 0 0)
   )
-  (junction (at 109.22 143.51) (diameter 0) (color 0 0 0 0)
-  )
   (junction (at 212.09 55.88) (diameter 0) (color 0 0 0 0)
   )
@@
   )
   (junction (at 177.8 121.92) (diameter 0) (color 0 0 0 0)
-  )
-  (junction (at 127 158.75) (diameter 0) (color 0 0 0 0)
   )
   (junction (at 172.72 52.07) (diameter 0) (color 0 0 0 0)
@@
     (stroke (width 0) (type default) (color 0 0 0 0))
   )
-  (wire (pts (xy 124.46 134.62) (xy 127 134.62))
-    (stroke (width 0) (type default) (color 0 0 0 0))
-  )
   (wire (pts (xy 114.3 71.12) (xy 118.11 71.12))
     (stroke (width 0) (type default) (color 0 0 0 0))
@@
     (stroke (width 0) (type default) (color 0 0 0 0))
   )
-  (wire (pts (xy 127 158.75) (xy 129.54 158.75))
-    (stroke (width 0) (type default) (color 0 0 0 0))
-  )
   (wire (pts (xy 120.65 68.58) (xy 120.65 72.39))
     (stroke (width 0) (type default) (color 0 0 0 0))
   )
-  (wire (pts (xy 109.22 143.51) (xy 109.22 134.62))
-    (stroke (width 0) (type default) (color 0 0 0 0))
-  )
   (wire (pts (xy 190.5 52.07) (xy 189.23 52.07))
     (stroke (width 0) (type default) (color 0 0 0 0))
@@
     (stroke (width 0) (type default) (color 0 0 0 0))
   )
-  (wire (pts (xy 116.84 167.64) (xy 127 167.64))
-    (stroke (width 0) (type default) (color 0 0 0 0))
-  )
   (wire (pts (xy 116.84 55.88) (xy 116.84 68.58))
     (stroke (width 0) (type default) (color 0 0 0 0))
@@
     (stroke (width 0) (type default) (color 0 0 0 0))
   )
-  (wire (pts (xy 124.46 158.75) (xy 127 158.75))
-    (stroke (width 0) (type default) (color 0 0 0 0))
-  )
   (wire (pts (xy 49.53 163.83) (xy 49.53 166.37))
     (stroke (width 0) (type default) (color 0 0 0 0))
@@
     (stroke (width 0) (type default) (color 0 0 0 0))
   )
-  (wire (pts (xy 111.76 143.51) (xy 109.22 143.51))
-    (stroke (width 0) (type default) (color 0 0 0 0))
-  )
   (bus (pts (xy 173.99 92.71) (xy 173.99 97.79))
     (stroke (width 0) (type default) (color 0 0 0 0))
@@
     (stroke (width 0) (type default) (color 0 0 0 0))
   )
-  (wire (pts (xy 127 134.62) (xy 129.54 134.62))
-    (stroke (width 0) (type default) (color 0 0 0 0))
-  )
-  (wire (pts (xy 127 143.51) (xy 127 134.62))
-    (stroke (width 0) (type default) (color 0 0 0 0))
-  )
   (wire (pts (xy 83.82 55.88) (xy 87.63 55.88))
     (stroke (width 0) (type default) (color 0 0 0 0))
@@
     (stroke (width 0) (type default) (color 0 0 0 0))
   )
-  (wire (pts (xy 127 167.64) (xy 127 158.75))
-    (stroke (width 0) (type default) (color 0 0 0 0))
-  )
   (wire (pts (xy 102.87 64.77) (xy 114.3 64.77))
     (stroke (width 0) (type default) (color 0 0 0 0))
@@
     (stroke (width 0) (type default) (color 0 0 0 0))
   )
-  (wire (pts (xy 116.84 143.51) (xy 127 143.51))
-    (stroke (width 0) (type default) (color 0 0 0 0))
-  )
   (wire (pts (xy 63.5 163.83) (xy 63.5 166.37))
     (stroke (width 0) (type default) (color 0 0 0 0))
@@
     (stroke (width 0) (type default) (color 0 0 0 0))
   )
-  (wire (pts (xy 111.76 167.64) (xy 109.22 167.64))
-    (stroke (width 0) (type default) (color 0 0 0 0))
-  )
   (wire (pts (xy 120.65 72.39) (xy 134.62 72.39))
     (stroke (width 0) (type default) (color 0 0 0 0))
@@
     (stroke (width 0) (type default) (color 0 0 0 0))
   )
-  (wire (pts (xy 109.22 167.64) (xy 109.22 158.75))
-    (stroke (width 0) (type default) (color 0 0 0 0))
-  )
   (wire (pts (xy 189.23 52.07) (xy 182.88 52.07))
     (stroke (width 0) (type default) (color 0 0 0 0))
@@
     (effects (font (size 1.27 1.27)) (justify left bottom))
   )
-  (label "FTRIG" (at 129.54 158.75 0)
-    (effects (font (size 1.27 1.27)) (justify left bottom))
-  )
   (label "GND" (at 165.1 113.03 0)
     (effects (font (size 1.27 1.27)) (justify left bottom))
@@
   )
   (label "RST" (at 127 100.33 0)
-    (effects (font (size 1.27 1.27)) (justify left bottom))
-  )
-  (label "STRIG" (at 129.54 134.62 0)
     (effects (font (size 1.27 1.27)) (justify left bottom))
   )
@@
     (pin "2")
   )
-  (symbol (lib_id "Device:C_Small") (at 114.3 167.64 270) (unit 1)
-    (in_bom yes) (on_board yes) (fields_autoplaced)
-    (property "Reference" "C6" (id 0) (at 114.2936 161.29 90))
-    (property "Value" "0u1" (id 1) (at 114.2936 163.83 90))
-    (property "Footprint" "Capacitor_SMD:C_0603_1608Metric_Pad1.08x0.95mm_HandSolder" (id 2) (at 114.3 167.64 0)
-      (effects (font (size 1.27 1.27)) hide)
-    )
-    (property "Datasheet" "~" (id 3) (at 114.3 167.64 0)
-      (effects (font (size 1.27 1.27)) hide)
-    )
-    (pin "1")
-    (pin "2")
-  )
-  (symbol (lib_id "power:GND") (at 109.22 143.51 0) (unit 1)
-    (in_bom yes) (on_board yes) (fields_autoplaced)
-    (property "Reference" "#PWR013" (id 0) (at 109.22 149.86 0)
-      (effects (font (size 1.27 1.27)) hide)
-    )
-    (property "Value" "GND" (id 1) (at 109.22 148.59 0))
-    (property "Footprint" "" (id 2) (at 109.22 143.51 0)
-      (effects (font (size 1.27 1.27)) hide)
-    )
-    (property "Datasheet" "" (id 3) (at 109.22 143.51 0)
-      (effects (font (size 1.27 1.27)) hide)
-    )
-    (pin "1")
-  )
   (symbol (lib_id "Device:R_Small") (at 100.33 55.88 90) (unit 1)
     (in_bom yes) (on_board yes) (fields_autoplaced)
@@
     )
     (property "Datasheet" "~" (id 3) (at 100.33 55.88 0)
-      (effects (font (size 1.27 1.27)) hide)
-    )
-    (pin "1")
-    (pin "2")
-  )
-  (symbol (lib_id "Device:C_Small") (at 114.3 143.51 270) (unit 1)
-    (in_bom yes) (on_board yes) (fields_autoplaced)
-    (property "Reference" "C5" (id 0) (at 114.2936 137.16 90))
-    (property "Value" "0u1" (id 1) (at 114.2936 139.7 90))
-    (property "Footprint" "Capacitor_SMD:C_0603_1608Metric_Pad1.08x0.95mm_HandSolder" (id 2) (at 114.3 143.51 0)
-      (effects (font (size 1.27 1.27)) hide)
-    )
-    (property "Datasheet" "~" (id 3) (at 114.3 143.51 0)
       (effects (font (size 1.27 1.27)) hide)
     )
@@
     (pin "2")
   )
-  (symbol (lib_id "4-1437565-2:4-1437565-2") (at 116.84 134.62 0) (unit 1)
-    (in_bom yes) (on_board yes) (fields_autoplaced)
-    (property "Reference" "S3" (id 0) (at 116.84 127 0))
-    (property "Value" "4-1437565-2" (id 1) (at 116.84 129.54 0))
-    (property "Footprint" "footprint:SW_4-1437565-2" (id 2) (at 116.84 134.62 0)
-      (effects (font (size 1.27 1.27)) (justify bottom) hide)
-    )
-    (property "Datasheet" "" (id 3) (at 116.84 134.62 0)
-      (effects (font (size 1.27 1.27)) hide)
-    )
-    (property "EU_RoHS_Compliance" "Compliant" (id 4) (at 116.84 134.62 0)
-      (effects (font (size 1.27 1.27)) (justify bottom) hide)
-    )
-    (property "Comment" "4-1437565-2" (id 5) (at 116.84 134.62 0)
-      (effects (font (size 1.27 1.27)) (justify bottom) hide)
-    )
-    (pin "1")
-    (pin "2")
-    (pin "3")
-    (pin "4")
-  )
   (symbol (lib_id "Device:R_Small") (at 49.53 161.29 0) (unit 1)
     (in_bom yes) (on_board yes) (fields_autoplaced)
@@
     (pin "2")
   )
-  (symbol (lib_id "power:GND") (at 109.22 167.64 0) (unit 1)
-    (in_bom yes) (on_board yes) (fields_autoplaced)
-    (property "Reference" "#PWR014" (id 0) (at 109.22 173.99 0)
-      (effects (font (size 1.27 1.27)) hide)
-    )
-    (property "Value" "GND" (id 1) (at 109.22 172.72 0))
-    (property "Footprint" "" (id 2) (at 109.22 167.64 0)
-      (effects (font (size 1.27 1.27)) hide)
-    )
-    (property "Datasheet" "" (id 3) (at 109.22 167.64 0)
-      (effects (font (size 1.27 1.27)) hide)
-    )
-    (pin "1")
-  )
   (symbol (lib_id "Device:C_Small") (at 85.09 167.64 270) (unit 1)
     (in_bom yes) (on_board yes) (fields_autoplaced)
@@
     (pin "2")
   )
-  (symbol (lib_id "4-1437565-2:4-1437565-2") (at 116.84 158.75 0) (unit 1)
-    (in_bom yes) (on_board yes)
-    (property "Reference" "S4" (id 0) (at 116.84 151.13 0))
-    (property "Value" "4-1437565-2" (id 1) (at 116.84 153.67 0))
-    (property "Footprint" "footprint:SW_4-1437565-2" (id 2) (at 116.84 158.75 0)
-      (effects (font (size 1.27 1.27)) (justify bottom) hide)
-    )
-    (property "Datasheet" "" (id 3) (at 116.84 158.75 0)
-      (effects (font (size 1.27 1.27)) hide)
-    )
-    (property "EU_RoHS_Compliance" "Compliant" (id 4) (at 116.84 158.75 0)
-      (effects (font (size 1.27 1.27)) (justify bottom) hide)
-    )
-    (property "Comment" "4-1437565-2" (id 5) (at 116.84 158.75 0)
-      (effects (font (size 1.27 1.27)) (justify bottom) hide)
-    )
-    (pin "1")
-    (pin "2")
-    (pin "3")
-    (pin "4")
-  )
   (symbol (lib_id "power:GND") (at 83.82 76.2 0) (unit 1)
